File: EAGLE/StandingDesk/untitled.brd (EAGLE design)
At the start: 84.4 x 51.1 mm, 39 parts, among them IC1 ISL21080, J1 39301060, J2 1744429-2, U1 DRV8874PWPR, U2 LMV358

Commit message: Eagle work
Parts:
- moved C6 210.2 mm to (59.9, 26.4)
- moved C9 205.8 mm to (35.3, 22.1), turned to 270 degrees
- moved C8 202.8 mm to (42.7, 19.1), turned to 270 degrees
- moved C7 197.2 mm to (54.9, 6.86), turned to 270 degrees
- moved R18 186.3 mm to (35.6, 27.7), turned to 180 degrees
- moved R17 183.1 mm to (35.6, 29.7), turned to 180 degrees
- moved R16 179.8 mm to (35.6, 31.8), turned to 180 degrees
- moved R15 176.7 mm to (35.6, 33.8), turned to 180 degrees
- moved R14 173.5 mm to (35.6, 35.8), turned to 180 degrees
- moved R13 170.4 mm to (35.6, 37.8), turned to 180 degrees
- moved C4 168.8 mm to (39.4, 40.4)
- moved C5 168.5 mm to (35.3, 40.4), turned to 180 degrees
- moved J4 165.9 mm to (14.2, 12.2)
- moved IC1 165.1 mm to (37.3, 43.4)
- moved R12 156.0 mm to (49.8, 23.9), turned to 90 degrees
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Connections:
- net M_ONE: now also J1.5; no longer J1.4
- net M_TWO: now also J1.4; no longer J1.5
Routing:
- net VCC: track 0.00 -> 132.6 mm, vias 0 -> 3
- net 19V: track 0.00 -> 77.3 mm, vias 0 -> 2
- net PH/IN2: track 0.00 -> 59.6 mm
- net FAULT: track 0.00 -> 59.3 mm, vias 0 -> 2
- net SLEEP_IN: track 0.00 -> 59.2 mm
- net EN/IN1: track 0.00 -> 58.2 mm
- net GND: track 0.00 -> 43.4 mm, vias 0 -> 21
- net GPIO_2: track 0.00 -> 33.7 mm
- net BTN_2: track 0.00 -> 33.0 mm
- net ISENSE: track 0.00 -> 29.6 mm
- net BTN_1: track 0.00 -> 28.2 mm
- net GPIO_2_PROTECTED: track 0.00 -> 26.1 mm
- net VREF: track 0.00 -> 19.5 mm
- net GPIO_1: track 0.00 -> 17.1 mm
- net N$8: track 0.00 -> 15.3 mm
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- added copper zone on layer 16, net GND
- added copper zone on layer 1, net M_ONE
- added copper zone on layer 1, net M_TWO
Other:
- board size 84.4 x 51.1 mm -> 85.1 x 50 mm
- board text added: "19V"
- board text added: "BTN1"
- board text added: "BTN2"
- board text added: "GND"
- board text added: "VCC"
