File: EAGLE/StandingDesk/untitled.sch (EAGLE design)
At the start: 39 parts, among them IC1 ISL21080, J1 39301060, J2 1744429-2, U1 DRV8874PWPR, U2 LMV358

Commit message: Eagle work
Connections:
- net M_ONE: now also J1.5; no longer J1.4
- net M_TWO: now also J1.4; no longer J1.5
Changed lines of the file:
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@@
 <net name="M_ONE" class="0">
+<segment>
+<pinref part="U1" gate="A" pin="OUT1"/>
+<wire x1="121.92" y1="111.76" x2="134.62" y2="111.76" width="0.1524" layer="91"/>
+<label x="127" y="111.76" size="1.778" layer="95"/>
+</segment>
+<segment>
+<pinref part="J1" gate="A" pin="5"/>
+<wire x1="302.26" y1="101.6" x2="281.94" y2="101.6" width="0.1524" layer="91"/>
+<label x="281.94" y="101.6" size="1.778" layer="95"/>
+</segment>
+</net>
+<net name="M_TWO" class="0">
+<segment>
+<pinref part="U1" gate="A" pin="OUT2"/>
+<wire x1="121.92" y1="96.52" x2="134.62" y2="96.52" width="0.1524" layer="91"/>
+<label x="127" y="96.52" size="1.778" layer="95"/>
+</segment>
 <segment>
 <pinref part="J1" gate="A" pin="4"/>
 <wire x1="302.26" y1="104.14" x2="281.94" y2="104.14" width="0.1524" layer="91"/>
 <label x="281.94" y="104.14" size="1.778" layer="95"/>
-</segment>
-<segment>
-<pinref part="U1" gate="A" pin="OUT1"/>
-<wire x1="121.92" y1="111.76" x2="134.62" y2="111.76" width="0.1524" layer="91"/>
-<label x="127" y="111.76" size="1.778" layer="95"/>
-</segment>
-</net>
-<net name="M_TWO" class="0">
-<segment>
-<pinref part="J1" gate="A" pin="5"/>
-<wire x1="302.26" y1="101.6" x2="281.94" y2="101.6" width="0.1524" layer="91"/>
-<label x="281.94" y="101.6" size="1.778" layer="95"/>
-</segment>
-<segment>
-<pinref part="U1" gate="A" pin="OUT2"/>
-<wire x1="121.92" y1="96.52" x2="134.62" y2="96.52" width="0.1524" layer="91"/>
-<label x="127" y="96.52" size="1.778" layer="95"/>
 </segment>
 </net>
@@
 </sheet>
 </sheets>
+<errors>
+</errors>
 </schematic>
 </drawing>
