File: EAGLE/StandingDesk V1/untitled.brd (EAGLE design)
At the start: 85.1 x 50 mm, 39 parts, among them IC1 ISL21080, J1 39301060, J2 1744429-2, U1 DRV8874PWPR, U2 LMV358

Commit message: Finally adding everything else
Parts:
- IC1: value ISL21080 -> ISL21080DIH310Z-TK
- moved J3 16.8 mm to (32.5, 13.5)
Routing:
- net VCC: track 137.3 -> 183.8 mm
- net 19V: track 60.7 -> 77.3 mm
- net VREF: track 18.5 -> 19.5 mm
Other:
- board text added: "19V"
- board text added: "BTN1"
- board text added: "BTN2"
- board text added: "GND"
- board text added: "VCC"
